File: Electrical/LCP_Controller/ADC_24Bit.kicad_sch (KiCad schematic)
At the start: 17 parts, among them Q1 TSM500P02CX RFG, U1 ADS1219

Commit message: Hardware Revision : v0.3
1. modified schematic design, removed unnecessary test points.
2. pcb layout 2x8 Inches allowance dimension, layout is in progress
Parts:
- removed RN1: 2k2, Resistor_SMD:R_Array_Concave_2x0603, symbol Device:R_Pack02
- removed TP14, TP15: 5002, TestPoint:TestPoint_Keystone_5000-5004_Miniature, symbol Connector:TestPoint
- removed TP16, TP7: 5004, TestPoint:TestPoint_Keystone_5000-5004_Miniature, symbol Connector:TestPoint
- removed TP17, TP18: 5001, TestPoint:TestPoint_Keystone_5000-5004_Miniature, symbol Connector:TestPoint
- renumbered C2 to C27, C3 to C28, C1 to C29, JP1 to JP5, JP2 to JP6, JP3 to JP7, Q1 to Q7, R1 to R21, RN2 to RN5, U1 to U8
