File: Electrical/LCP_Controller/COM0_COM1.kicad_sch (KiCad schematic)
At the start: 23 parts, among them J2 SALEAE_TEST, J3 SALEAE_TEST, Q4 TSM500P02CX RFG, Q5 TSM500P02CX RFG, U6 TRS3122E

Commit message: Hardware Revision : v0.3
1. modified schematic design, removed unnecessary test points.
2. pcb layout 2x8 Inches allowance dimension, layout is in progress
Parts:
- removed J2, J3: SALEAE_TEST, Connector_PinHeader_2.54mm:PinHeader_2x04_P2.54mm_Vertical, symbol Connector_Generic:Conn_02x04_Odd_Even
- removed TP33, TP34: 5002, TestPoint:TestPoint_Keystone_5000-5004_Miniature, symbol Connector:TestPoint
- removed TP35, TP36: 5001, TestPoint:TestPoint_Keystone_5000-5004_Miniature, symbol Connector:TestPoint
- removed TP37, TP38: 5004, TestPoint:TestPoint_Keystone_5000-5004_Miniature, symbol Connector:TestPoint
- renumbered C21 to C38, C18 to C39, C23 to C40, C19 to C41, C22 to C42, C20 to C43, Q4 to Q10, Q5 to Q11, R13 to R24, R14 to R25, RN5 to RN6, RN6 to RN7, RN7 to RN8, RN8 to RN9, U6 to U11
Connections:
- no-connect marks 2 -> 0

Commit message: Hw Rev : 0.3v updated
changed TRS3122ERGER to TRS3122ERGET due to shortage of part.
Parts:
- RN6, RN7, RN8, RN9: footprint Resistor_SMD:R_Array_Concave_2x0603 -> Resistor_SMD:R_Array_Convex_2x0402
- U11: MPN TRS3122ERGER -> TRS3122ERGET
Changed lines of the file:
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@@
     (property "Reference" "RN6" (id 0) (at 127 56.7182 90))
     (property "Value" "Jumper/0Ohm" (id 1) (at 127 59.0296 90))
-    (property "Footprint" "Resistor_SMD:R_Array_Concave_2x0603" (id 2) (at 127 69.215 90)
+    (property "Footprint" "Resistor_SMD:R_Array_Convex_2x0402" (id 2) (at 127 69.215 90)
       (effects (font (size 1.27 1.27)) hide)
     )
@@
     (property "Reference" "RN7" (id 0) (at 127 68.1482 90))
     (property "Value" "Jumper/0Ohm" (id 1) (at 127 70.4596 90))
-    (property "Footprint" "Resistor_SMD:R_Array_Concave_2x0603" (id 2) (at 127 80.645 90)
+    (property "Footprint" "Resistor_SMD:R_Array_Convex_2x0402" (id 2) (at 127 80.645 90)
       (effects (font (size 1.27 1.27)) hide)
     )
@@
     (property "Reference" "RN9" (id 0) (at 127 116.4082 90))
     (property "Value" "Jumper/0Ohm" (id 1) (at 127 118.7196 90))
-    (property "Footprint" "Resistor_SMD:R_Array_Concave_2x0603" (id 2) (at 127 128.905 90)
+    (property "Footprint" "Resistor_SMD:R_Array_Convex_2x0402" (id 2) (at 127 128.905 90)
       (effects (font (size 1.27 1.27)) hide)
     )
@@
     (property "Reference" "RN8" (id 0) (at 127 104.9782 90))
     (property "Value" "Jumper/0Ohm" (id 1) (at 127 107.2896 90))
-    (property "Footprint" "Resistor_SMD:R_Array_Concave_2x0603" (id 2) (at 127 117.475 90)
+    (property "Footprint" "Resistor_SMD:R_Array_Convex_2x0402" (id 2) (at 127 117.475 90)
       (effects (font (size 1.27 1.27)) hide)
     )
@@
       (effects (font (size 1.27 1.27)) hide)
     )
-    (property "MPN" "TRS3122ERGER" (id 4) (at 189.23 64.77 0)
+    (property "MPN" "TRS3122ERGET" (id 4) (at 189.23 64.77 0)
       (effects (font (size 1.27 1.27)) hide)
     )
