File: Electrical/LCP_Controller/COM2_COM3.kicad_sch (KiCad schematic)
At the start: 39 parts, among them J4 SALEAE_TEST, J5 SALEAE_TEST, Q6 TSM500P02CX RFG, Q7 TSM500P02CX RFG, U7 SN55HVD75-EP, U8 SN55HVD75-EP, U9 TRS3122E

Commit message: Hardware Revision : v0.3
1. modified schematic design, removed unnecessary test points.
2. pcb layout 2x8 Inches allowance dimension, layout is in progress
Parts:
- removed D4, D5: CDSOT23-SM712, Package_TO_SOT_SMD:SOT-23, symbol Device:D_TVS_x2_AAC
- removed J4, J5: SALEAE_TEST, Connector_PinHeader_2.54mm:PinHeader_2x04_P2.54mm_Vertical, symbol Connector_Generic:Conn_02x04_Odd_Even
- removed TP39, TP40: 5001, TestPoint:TestPoint_Keystone_5000-5004_Miniature, symbol Connector:TestPoint
- removed TP41, TP42: 5002, TestPoint:TestPoint_Keystone_5000-5004_Miniature, symbol Connector:TestPoint
- removed TP43, TP44: 5004, TestPoint:TestPoint_Keystone_5000-5004_Miniature, symbol Connector:TestPoint
- added D5, D6: CDSOT23-SM712, Package_TO_SOT_SMD:SOT-23, symbol Device:D_TVS_Dual_AAC
- renumbered C29 to C44, C26 to C45, C31 to C46, C27 to C47, C30 to C48, C28 to C49, C24 to C50, C25 to C51, Q6 to Q12, Q7 to Q13, R17 to R26, R21 to R27, R18 to R28, R19 to R29, R22 to R30, R20 to R31, R15 to R32, R16 to R33, RN9 to RN10, RN10 to RN11, RN11 to RN12, RN12 to RN13, RN15 to RN14, RN13 to RN15, RN14 to RN17, U9 to U12, U7 to U13, U8 to U14
Connections:
- net COM2_RX(D-): now also D5.2 (A2)
- net COM2_TX(D+): now also D5.1 (A1)
- net COM3_RX(D-): now also D6.2 (A2)
- net COM3_TX(D+): now also D6.1 (A1)
- net GND: now also D5.3 (common), D6.3 (common)
- no-connect marks 14 -> 12

Commit message: Hw Rev : 0.3v updated
changed TRS3122ERGER to TRS3122ERGET due to shortage of part.
Parts:
- U12: MPN TRS3122ERGER -> TRS3122ERGET
Changed lines of the file:
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@@
       (effects (font (size 1.27 1.27)) hide)
     )
-    (property "MPN" "TRS3122ERGER" (id 4) (at 246.38 113.03 0)
+    (property "MPN" "TRS3122ERGET" (id 4) (at 246.38 113.03 0)
       (effects (font (size 1.27 1.27)) hide)
     )
