File: Electrical/LCP_Controller/Connectors.kicad_sch (KiCad schematic)
At the start: 7 parts, among them J19 ANALOG_CONN, J20 Conn_01x04, J21 Conn_01x04, J22 Conn_01x04, J23 Conn_01x04, J24 Conn_01x04, J25 Conn_01x04

Commit message: Removed the rest of the test ports
Layout updates
Parts:
- J19: footprint Connector_PinHeader_2.54mm:PinHeader_2x04_P2.54mm_Vertical -> Connector_Molex:Molex_Micro-Fit_3.0_43045-0812_2x04_P3.00mm_Vertical
Changed lines of the file:
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@@
       (effects (font (size 1.27 1.27)) (justify right))
     )
-    (property "Footprint" "Connector_PinHeader_2.54mm:PinHeader_2x04_P2.54mm_Vertical" (at 171.45 46.99 0)
+    (property "Footprint" "Connector_Molex:Molex_Micro-Fit_3.0_43045-0812_2x04_P3.00mm_Vertical" (at 171.45 46.99 0)
       (effects (font (size 1.27 1.27)) hide)
     )
